File: MAIN PCB/ADSR Main Pcb.kicad_pcb (KiCad board)
At the start: 2 copper layers, 98 x 164 mm, 81 parts, among them J9 POWER, Q1 2N3904, Q2 2N3904, Q3 2N3904, Q4 2N3904, U1 ENV GEN 8C, U2 ENV GEN 8C, U3 ENV GEN 8C, U4 ENV GEN 8C, U5 TL074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

Commit message: Add files via upload
Routing:
- net Net-(U6A--): track 4.68 -> 7.68 mm
Changed lines of the file:
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@@
   (segment (start 83.75 70.77) (end 83.75 67.14) (width 0.5) (layer "F.Cu") (net 38))
   (segment (start 83.75 67.14) (end 85.19 65.7) (width 0.5) (layer "F.Cu") (net 38))
+  (segment (start 92.81 62.7) (end 92.81 65.7) (width 0.5) (layer "F.Cu") (net 39))
   (segment (start 92.81 62.7) (end 96.5 62.7) (width 0.5) (layer "F.Cu") (net 39))
   (segment (start 96.5 62.7) (end 97.2 62) (width 0.5) (layer "F.Cu") (net 39))
